File: HALMET.kicad_pcb (KiCad board)
At the start: 4 copper layers, 89 x 58 mm, 251 parts, among them J1103 Conn_01x02, J1104 Conn_01x02, J1105 Conn_01x02, J1106 Conn_01x02, J1201 Conn_01x02, J201 GPIO, J203 Conn_01x01, J302 Conn_01x02, J401 USB_B_Micro, J402 Conn_01x04, J501 EXT LEDS, J602 Conn_02x04_Odd_Even, J604 Conn_01x02, J605 Conn_01x02, J606 Conn_01x02, J607 Conn_01x02, J702 Conn_01x04, J801 Conn_01x03, J802 Conn_01x04, Q401 S8050, Q402 S8050, Q601 BC856BW,115, Q602 BC856BW,115, Q603 BC856BW,115, Q604 BC856BW,115, SW501 SW_Push, SW502 SW_Push, U1101 74LVC1G17, U1102 74LVC1G17, U1103 74LVC1G17, U1104 74LVC1G17, U1200 ICM-42688-P, U1201 π140U30, U1202 ISO1540, U1203 XC6206P332MR, U201 ESP32-S3-WROOM-1U-N16R2, U202 XL1509-3.3, U203 LM317L_SOT-89, U401 CH340C, U402 USBLC6-2SC6, U501 SN65HVD230DR, U502 SP3485EN, U601 LMV324, U602 ADS1115IDGS

Commit message: Updated LCSC part numbers
Parts:
- R504: value 1k -> 75R
- R505: value 1k -> 240R
- U201: value ESP32-S3-WROOM-1U-N16R2 -> ESP32-S3-WROOM-1U-N16R8

Commit message: Moved ESP32-S3 + larger pin headers
Parts:
- J501: footprint Connector_PinHeader_1.00mm:PinHeader_1x03_P1.00mm_Vertical -> Connector_PinHeader_2.00mm:PinHeader_1x03_P2.00mm_Vertical
- JP1: footprint Connector_PinHeader_1.00mm:PinHeader_1x02_P1.00mm_Vertical -> Connector_PinHeader_2.00mm:PinHeader_1x02_P2.00mm_Vertical
- moved U201 0.75 mm to (161.4, 76.0)
- moved REF** 0.69 mm to (123.3, 97.5)
- moved J501 0.58 mm to (114.3, 103.0)
- moved C616 0.46 mm to (172.7, 75.5)
- moved CR501 0.46 mm to (175.7, 74.9)
- moved F501 0.46 mm to (174.7, 71.1)
- moved F502 0.46 mm to (174.6, 67.2)
- moved U502 0.46 mm to (174.7, 80.5)
- moved R403 0.33 mm to (172.6, 86.9)
- moved R404 0.33 mm to (172.6, 85.0)
- moved U402 0.33 mm to (175.4, 85.9)
- moved C203 0.32 mm to (169.3, 87.5)
- moved R201 0.32 mm to (170.4, 87.6)
- moved JP1 0.18 mm to (149.0, 84.9), turned to 180 degrees
Routing:
- net /UART0_RX: track 8.78 -> 12.1 mm
- net /UART0_TX: track 11.5 -> 9.14 mm
- net GND: track 165.6 -> 163.3 mm, vias 78 -> 76
- net /User Interface/<NO NET>: track 31.9 -> 29.8 mm, vias 2 -> 1
- net /SCL: track 97.6 -> 95.8 mm, vias 8 -> 6
- net /DI2: track 12.1 -> 10.7 mm
- net /USB_D_MINUS: track 27.8 -> 29.0 mm
- net /SDA: track 91.7 -> 90.6 mm, vias 7 -> 5
- net Net-(J501-Pin_2): track 21.3 -> 20.2 mm, vias 2 -> 1
- net /CAN_L: track 49.1 -> 50.2 mm
- net /DI3: track 11.8 -> 10.7 mm
- net /USB_D_PLUS: track 30.1 -> 31.1 mm
- net /UART1_RX: track 23.7 -> 24.7 mm
- net /ESP32/IO0: track 13.8 -> 12.8 mm
- net /ESP32/IO4: track 23.5 -> 22.6 mm
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Other:
- board text added: "Nav Core Processor"
- board text added: "□6.4V ■5.0V"
- board text removed: "Marine Sensor & Compute Module"
- board text removed: "Ø→6.4V MHU J→5V"
