File: PCB.kicad_sch (KiCad schematic)
At the start: 8 parts

Commit message: Initial V1.0.0 Bluefin forked
Added ICM-42688-P 6-axis IMU
Added LM317 LDO for 6.4v or 5v MHU supply (selectable via jumper)
Added External LED's for IO2 (Pin 24) and 3.3v
Parts:
- removed G605: HL-Logo, HALMET:Hat_Labs_25.4mm, symbol Graphic:SYM_Radioactive_Radiation_Small
- removed G701: HL-Pictogram, HALMET:HaL_picto_8mm, symbol Graphic:SYM_Radioactive_Radiation_Small
Changed lines of the file:
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@@
-	(symbol
-		(lib_id "Graphic:SYM_Radioactive_Radiation_Small")
-		(at 160.02 82.55 0)
-		(unit 1)
-		(exclude_from_sim yes)
-		(in_bom no)
-		(on_board yes)
-		(dnp no)
-		(fields_autoplaced yes)
-		(property "Reference" "G605"
-			(at 163.83 80.9625 0)
-			(effects
-				(font
-					(size 1.27 1.27)
-				)
-				(justify left)
-			)
-		)
-		(property "Value" "HL-Logo"
-			(at 163.83 83.5025 0)
-			(effects
-				(font
-					(size 1.27 1.27)
-				)
-				(justify left)
-			)
-		)
-		(property "Footprint" "HALMET:Hat_Labs_25.4mm"
-			(at 160.02 82.55 0)
-			(effects
-				(font
-					(size 1.27 1.27)
-				)
-				(hide yes)
-			)
-		)
-		(property "Datasheet" "~"
-			(at 160.782 87.63 0)
-			(effects
-				(font
-					(size 1.27 1.27)
-				)
-				(hide yes)
-			)
-		)
-		(property "Description" ""
-			(at 160.02 82.55 0)
-			(effects
-				(font
-					(size 1.27 1.27)
-				)
-			)
-		)
-		(instances
-			(project "HALMET"
-				(path "/dff502f1-2fe5-4c09-a767-aabc78c2e052/00000000-0000-0000-0000-00005fc0c355"
-					(reference "G605")
-					(unit 1)
-				)
-			)
-		)
-	)
 	(symbol
 		(lib_id "Graphic:SYM_Radioactive_Radiation_Small")
@@
 					(unit 1)
 				)
-			)
-		)
-	)
-	(symbol
-		(lib_id "Graphic:SYM_Radioactive_Radiation_Small")
-		(at 160.02 91.44 0)
-		(unit 1)
-		(exclude_from_sim yes)
-		(in_bom no)
-		(on_board yes)
-		(dnp no)
-		(fields_autoplaced yes)
-		(property "Reference" "G701"
-			(at 163.83 89.8525 0)
-			(effects
-				(font
-					(size 1.27 1.27)
-				)
-				(justify left)
-			)
-		)
-		(property "Value" "HL-Pictogram"
-			(at 163.83 92.3925 0)
-			(effects
-				(font
-					(size 1.27 1.27)
-				)
-				(justify left)
-			)
-		)
-		(property "Footprint" "HALMET:HaL_picto_8mm"
-			(at 160.02 91.44 0)
-			(effects
-				(font
-					(size 1.27 1.27)
-				)
-				(hide yes)
-			)
-		)
-		(property "Datasheet" "~"
-			(at 160.782 96.52 0)
-			(effects
-				(font
-					(size 1.27 1.27)
-				)
-				(hide yes)
-			)
-		)
-		(property "Description" ""
-			(at 160.02 91.44 0)
-			(effects
-				(font
-					(size 1.27 1.27)
-				)
-			)
-		)
-		(instances
-			(project "HALMET"
-				(path "/dff502f1-2fe5-4c09-a767-aabc78c2e052/00000000-0000-0000-0000-00005fc0c355"
-					(reference "G701")
-					(unit 1)
-				)

Commit message: Moved ESP32-S3 + larger pin headers
Other:
- company: Hat Labs Ltd -> Fifty One North Limited
- title: Hat Labs Marine Engine & Tank interface (HALMET) -> Bluefin Marine Processor
Changed lines of the file:
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@@
 	(paper "A4")
 	(title_block
-		(title "Hat Labs Marine Engine & Tank interface (HALMET)")
-		(date "2024-01-18")
-		(rev "1.0.1")
-		(company "Hat Labs Ltd")
-		(comment 1 "https://creativecommons.org/licenses/by-sa/4.0")
-		(comment 2 "To view a copy of this license, visit ")
-		(comment 3 "HALMET is licensed under CC BY-SA 4.0.")
+		(title "Bluefin Marine Processor")
+		(date "2026-01-08")
+		(rev "1.0.0")
+		(company "Fifty One North Limited")
+		(comment 1 "https://creativecommons.org/licenses/by-sa/4.0/")
+		(comment 2 "Bluefin is licensed under CC BY-SA 4.0")
+		(comment 3 "Modifications © 2026 Fiftyone North Ltd.")
+		(comment 4 "Based on an original design by Hat Labs Ltd.")
 	)
 	(text "Mounting holes"
