File: isolation.kicad_sch (KiCad schematic)
At the start: 20 parts, among them J1201 Conn_01x02, U1201 π140U30, U1202 ISO1540, U1203 XC6206P332MR

Commit message: Moved ESP32-S3 + larger pin headers
Other:
- company: Hat Labs Ltd -> Fifty One North Limited
- title: Hat Labs Marine Engine & Tank interface (HALMET) -> Bluefin Marine Processor
Changed lines of the file:
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@@
 	(paper "A4")
 	(title_block
-		(title "Hat Labs Marine Engine & Tank interface (HALMET)")
-		(date "2024-01-18")
-		(rev "1.0.1")
-		(company "Hat Labs Ltd")
-		(comment 1 "https://creativecommons.org/licenses/by-sa/4.0")
-		(comment 2 "To view a copy of this license, visit ")
-		(comment 3 "HALMET is licensed under CC BY-SA 4.0.")
+		(title "Bluefin Marine Processor")
+		(date "2026-01-08")
+		(rev "1.0.0")
+		(company "Fifty One North Limited")
+		(comment 1 "https://creativecommons.org/licenses/by-sa/4.0/")
+		(comment 2 "Bluefin is licensed under CC BY-SA 4.0")
+		(comment 3 "Modifications © 2026 Fiftyone North Ltd.")
+		(comment 4 "Based on an original design by Hat Labs Ltd.")
 	)
 	(text "Dummy load to help \nwith load regulation"
