File: serial.kicad_sch (KiCad schematic)
At the start: 12 parts, among them U501 SN65HVD230DR, U502 SP3485EN

Commit message: Changed to ESP32-S3-WROOM-1U
Added ESP32-S3-WROOM-1U-N16R2  and updated all routing and pin assignments.

Added USB-OTG connected via JST-PH
Connections:
- net UART1_RX renamed RS485_TX
- net UART1_TX renamed RS485_RX
Changed lines of the file:
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@@
 		)
 	)
-	(hierarchical_label "UART1_TX"
+	(hierarchical_label "RS485_RX"
 		(shape input)
 		(at 111.76 67.31 180)
@@
 		)
 	)
-	(hierarchical_label "UART1_RX"
+	(hierarchical_label "RS485_TX"
 		(shape output)
 		(at 111.76 57.15 180)

Commit message: Moved ESP32-S3 + larger pin headers
Other:
- company: Hat Labs Ltd -> Fifty One North Limited
- title: Hat Labs Marine Engine & Tank interface (HALMET) -> Bluefin Marine Processor
Changed lines of the file:
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@@
 	(paper "A4")
 	(title_block
-		(title "Hat Labs Marine Engine & Tank interface (HALMET)")
-		(date "2024-01-18")
-		(rev "1.0.1")
-		(company "Hat Labs Ltd")
-		(comment 1 "https://creativecommons.org/licenses/by-sa/4.0")
-		(comment 2 "To view a copy of this license, visit ")
-		(comment 3 "HALMET is licensed under CC BY-SA 4.0.")
+		(title "Bluefin Marine Processor")
+		(date "2026-01-08")
+		(rev "1.0.0")
+		(company "Fifty One North Limited")
+		(comment 1 "https://creativecommons.org/licenses/by-sa/4.0/")
+		(comment 2 "Bluefin is licensed under CC BY-SA 4.0")
+		(comment 3 "Modifications © 2026 Fiftyone North Ltd.")
+		(comment 4 "Based on an original design by Hat Labs Ltd.")
 	)
 	(text "Rs provides slope control\nto limit EMI."
